Commit message: adding new branch for Advanced Robotics

File: p3dx_description/urdf/pioneer3dx.xacro (robot description, xacro)
@@ -23,10 +23,5 @@
   <!-- chassis -->
 	<link name="base_link">
-		<inertial>
-			<mass value="3.5" />
-			<!--<origin xyz="-0.025 0 -0.223"/> -->
-			<origin xyz="-0.05 0 0" />
-			<inertia ixx="1" ixy="0" ixz="0" iyy="1" iyz="0" izz="1" />
-		</inertial>
+		<!--<inertial><mass value="3.5" /><!--<origin xyz="-0.025 0 -0.223"/> --><origin xyz="-0.05 0 0" /><inertia ixx="1" ixy="0" ixz="0" iyy="1" iyz="0" izz="1" /></inertial>-->
 		<visual name="base_visual">
 			<origin xyz="-0.045 0 0.148" rpy="0 0 0" />
